File: BenchBudEE.sch (KiCad schematic (older format))
At the start: 0 parts

Commit message: M3U5
Gah, forgot to sync the last one :)
Changed lines of the file:
@@
 LIBS:contrib
 LIBS:valves
+LIBS:BenchBudEEparts
 LIBS:BenchBudEE-cache
 EELAYER 27 0
@@
 Sheet 1 8
 Title ""
-Date "7 feb 2014"
+Date "10 feb 2014"
 Rev ""
 Comp ""
@@
 F5 "Tach_out" O L 6850 800 60
 F6 "Fan_in" I L 6850 950 60
+F7 "Current Measure" O L 6850 1800 60
+F8 "MOSI" I L 6850 1150 60
+F9 "MISO" O L 6850 1250 60
+F10 "CS_N" I L 6850 1450 60
+F11 "SCLK" I L 6850 1350 60
 $EndSheet
 $Sheet

Commit message: M3U6
Changed lines of the file:
@@
 $Descr A4 11693 8268
 encoding utf-8
-Sheet 1 8
+Sheet 1 9
 Title ""
 Date "10 feb 2014"
@@
 F1 "TerminalBlock.sch" 50
 $EndSheet
+$Sheet
+S 4800 1550 1700 1150
+U 52F9053E
+F0 "PowerAdjustmentMonitor" 50
+F1 "PowerAdjustmentMonitor.sch" 50
+$EndSheet
 $EndSCHEMATC
